File: sim/sim.sch (KiCad schematic (older format))
At the start: 4 parts, among them Q1 AO4407A

Commit message: sim
Parts:
- added D1: SS210, symbol Simulation_SPICE:DIODE
- added M1: MPMOS, symbol pspice:MPMOS
- added R2: 100k, symbol Device:R
- added R3: 100, symbol Device:R
- V1: value 5 -> 0 pwl(0US 0 99US 0 100US 5 199US 5 200US 0 499US 0 500US 5 799US 5 800US 0)
- V2: value sin(0 5 1k) -> 0 pwl(0US 0 299US 0 300US 3.2 399US 3.2 400US 0 599US 0 600US 3.2 699US 3.2 700US 0)
Connections:
- net GND: now also R2.1, R3.1
- removed net VCC: Q1.1 (S), Q1.2 (Sb), Q1.3 (Sc), V1.1 (E1)
- net VIN: no longer names the net of Q1.4 (G)
- net VIN: no longer V2.1 (E1)
- removed net Vload: Q1.5 (Dd), Q1.6 (Dc), Q1.7 (Db), Q1.8 (D), R1.1
- new net VBAT: M1.3 (S), M1.4 (B), V2.1 (E1)
- new net VLOAD: D1.2 (K), M1.1 (D), R1.1
- new net VUSB: D1.1 (A), R2.2, V1.1 (E1)
- new net Vg: M1.2 (G), R3.2
Other:
- note added: "1 Source; 8 Drain\n"
- moved on the sheet: Q1, R1, V1, V2
