File: sim/sim.sch (KiCad schematic (older format))
At the start: 8 parts, among them M1 MPMOS, Q1 AO4407A

Commit message: sim
Parts:
- removed D1: SS210, symbol Simulation_SPICE:DIODE
- removed Q1: AO4407A, Package_SO:SOIC-8_3.9x4.9mm_P1.27mm, symbol pace:AO4407A
- removed V1: 0 pwl(0US 0 99US 0 100US 5 199US 5 200US 0 499US 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, symbol pspice:VSOURCE
- added D1: DIODE, symbol pspice:DIODE
- added M2: MPMOS, symbol pspice:MPMOS
- added R4, R5, R6: 100k, symbol Device:R
- added V3: 0 sin(0, 5 , 1000), symbol pspice:VSOURCE
- M1: Spice_Lib_File (none) -> STD26P3LLH6.lib; Spice_Model (none) -> STD26P3LLH6; Spice_Netlist_Enabled (none) -> Y; Spice_Node_Sequence (none) -> 1 2 3; Spice_Primitive (none) -> X
- R2: value 100k -> .1
- V2: value 0 pwl(0US 0 299US 0 300US 3.2 399US 3.2 400US 0 599US 0 600US 3.2 699US 3.2 700US 0) -> 0 sin(0, 10, 2000, .0001)
Connections:
- net VUSB is gone; now on net VBAT: R2.2
- net GND: now also M2.2 (G), R4.1, R5.1, R6.1, V3.2 (E2); no longer R2.1, R3.1
- net VBAT: now also M1.1 (D), R5.2; no longer M1.3 (S), M1.4 (B), V2.1 (E1)
- net VLOAD: now also M2.3 (S), M2.4 (B); no longer M1.1 (D)
- net Vg: no longer names the net of M1.2 (G), R3.2
- new net: R2.1, V2.1 (E1)
- new net: D1.2 (A), M1.3 (S), M1.4 (B), M2.1 (D), R6.2
- new net Vusb: D1.1 (K), R3.1, R4.2, V3.1 (E1)
Other:
- note removed: "1 Source; 8 Drain\n"
- moved on the sheet: R1, R3, V2
