File: sim2/sim2.sch (KiCad schematic (older format))
At the start: 5 parts, among them M1 MNMOS

Commit message: sim
Parts:
- removed M1: MNMOS, symbol pspice:MNMOS
- added Q1: AO4407A, Package_SO:SOIC-8_3.9x4.9mm_P1.27mm, symbol pace:AO4407A
- added R?: 1k, symbol Device:R
Connections:
- net GND: now also R2.2, R?.2
- net Vg: now reaches R1.1
- net Vg: now also Q1.4 (G), R?.1
- net Vusb: now reaches R1.2, V2.1 (E1)
- net VCC renamed Vbat
- net Vbat: now also Q1.1 (S); no longer R2.1
- new net Vload: Q1.8 (D), R2.1
Other:
- moved on the sheet: R2
Changed lines of the file:
@@
 $EndDescr
-$Comp
-L pspice:MNMOS M1
-U 1 1 5F9ECAE3
-P 5850 3300
-F 0 "M1" H 6138 3346 50  0000 L CNN
-F 1 "MNMOS" H 6138 3255 50  0000 L CNN
-F 2 "" H 5825 3300 50  0001 C CNN
-F 3 "~" H 5825 3300 50  0001 C CNN
-	1    5850 3300
-	1    0    0    -1
-$EndComp
 $Comp
 L pspice:VSOURCE V1
@@
 $EndComp
 $Comp
-L power:VCC #PWR?
-U 1 1 5F9EDA7C
-P 2050 1650
-F 0 "#PWR?" H 2050 1500 50  0001 C CNN
-F 1 "VCC" H 2067 1823 50  0000 C CNN
-F 2 "" H 2050 1650 50  0001 C CNN
-F 3 "" H 2050 1650 50  0001 C CNN
-	1    2050 1650
-	1    0    0    -1
-$EndComp
-$Comp
-L power:GND #PWR?
+L power:GND #PWR02
 U 1 1 5F9EE039
 P 2050 2250
-F 0 "#PWR?" H 2050 2000 50  0001 C CNN
+F 0 "#PWR02" H 2050 2000 50  0001 C CNN
 F 1 "GND" H 2055 2077 50  0000 C CNN
 F 2 "" H 2050 2250 50  0001 C CNN
@@
 L Device:R R2
 U 1 1 5F9EE3C5
-P 5950 2800
-F 0 "R2" H 6020 2846 50  0000 L CNN
-F 1 "1k" H 6020 2755 50  0000 L CNN
-F 2 "" V 5880 2800 50  0001 C CNN
-F 3 "~" H 5950 2800 50  0001 C CNN
-	1    5950 2800
+P 6500 3950
+F 0 "R2" H 6570 3996 50  0000 L CNN
+F 1 "1k" H 6570 3905 50  0000 L CNN
+F 2 "" V 6430 3950 50  0001 C CNN
+F 3 "~" H 6500 3950 50  0001 C CNN
+	1    6500 3950
 	1    0    0    -1
 $EndComp
 $Comp
-L power:VCC #PWR?
-U 1 1 5F9EE8D9
-P 5950 2450
-F 0 "#PWR?" H 5950 2300 50  0001 C CNN
-F 1 "VCC" H 5967 2623 50  0000 C CNN
-F 2 "" H 5950 2450 50  0001 C CNN
-F 3 "" H 5950 2450 50  0001 C CNN
-	1    5950 2450
+L power:GND #PWR05
+U 1 1 5F9EED59
+P 6500 4350
+F 0 "#PWR05" H 6500 4100 50  0001 C CNN
+F 1 "GND" H 6505 4177 50  0000 C CNN
+F 2 "" H 6500 4350 50  0001 C CNN
+F 3 "" H 6500 4350 50  0001 C CNN
+	1    6500 4350
 	1    0    0    -1
 $EndComp
 Wire Wire Line
-	5950 2450 5950 2650
-Wire Wire Line
-	5950 2950 5950 3100
-$Comp
-L power:GND #PWR?
-U 1 1 5F9EED59
-P 5950 3750
-F 0 "#PWR?" H 5950 3500 50  0001 C CNN
-F 1 "GND" H 5955 3577 50  0000 C CNN
-F 2 "" H 5950 3750 50  0001 C CNN
-F 3 "" H 5950 3750 50  0001 C CNN
-	1    5950 3750
-	1    0    0    -1
-$EndComp
-Wire Wire Line
-	6050 3500 5950 3500
-Wire Wire Line
-	5950 3500 5950 3750
-Connection ~ 5950 3500
+	6500 4100 6500 4350
 $Comp
 L Device:R R1
@@
 $EndComp
 Wire Wire Line
-	5400 3300 5650 3300
+	5400 3300 5950 3300
 $Comp
 L pspice:VSOURCE V2
@@
 $EndComp
 $Comp
-L power:GND #PWR?
+L power:GND #PWR03
 U 1 1 5F9F1AC2
 P 4300 3900
-F 0 "#PWR?" H 4300 3650 50  0001 C CNN
+F 0 "#PWR03" H 4300 3650 50  0001 C CNN
 F 1 "GND" H 4305 3727 50  0000 C CNN
 F 2 "" H 4300 3900 50  0001 C CNN
@@
 Text Notes 4950 4500 0    50   ~ 0
 .tran 1us 1ms
+$Comp
+L pace:AO4407A Q1
+U 1 1 5F9EF2B4
+P 6400 3300
+F 0 "Q1" H 6605 3254 50  0000 L CNN
+F 1 "AO4407A" H 6605 3345 50  0000 L CNN
+F 2 "Package_SO:SOIC-8_3.9x4.9mm_P1.27mm" H 6600 3400 50  0001 C CNN
+F 3 "http://www.diodes.com/datasheets/AP1117.pdf" H 6400 3300 50  0001 C CNN
+F 4 "C16072" H 6400 3300 50  0001 C CNN "LCSC"
+F 5 "X" H 6400 3300 50  0001 C CNN "Spice_Primitive"
+F 6 "AO4407" H 6400 3300 50  0001 C CNN "Spice_Model"
+F 7 "Y" H 6400 3300 50  0001 C CNN "Spice_Netlist_Enabled"
+F 8 "/home/pace/eboard/sim/AO4407.mod" H 6400 3300 50  0001 C CNN "Spice_Lib_File"
+F 9 "8 4 1" H 6400 3300 50  0001 C CNN "Spice_Node_Sequence"
+	1    6400 3300
+	1    0    0    1
+$EndComp
+Wire Wire Line
+	6500 3800 6500 3500
+Wire Wire Line
+	6500 2450 6500 3100
+Text Label 4650 3300 0    50   ~ 0
+Vusb
+Text Label 5600 3300 0    50   ~ 0
+Vg
+Text Label 6500 3650 0    50   ~ 0
+Vload
+$Comp
+L Device:R R?
+U 1 1 5F9F9E7C
+P 5950 3950
+F 0 "R?" H 6020 3996 50  0000 L CNN
+F 1 "1k" H 6020 3905 50  0000 L CNN
+F 2 "" V 5880 3950 50  0001 C CNN
+F 3 "~" H 5950 3950 50  0001 C CNN
+	1    5950 3950
+	1    0    0    -1
+$EndComp
+Wire Wire Line
+	5950 3800 5950 3300
+Connection ~ 5950 3300
+Wire Wire Line
+	5950 3300 6200 3300
+$Comp
+L power:GND #PWR?
+U 1 1 5F9FA2FC
+P 5950 4350
+F 0 "#PWR?" H 5950 4100 50  0001 C CNN
+F 1 "GND" H 5955 4177 50  0000 C CNN
+F 2 "" H 5950 4350 50  0001 C CNN
+F 3 "" H 5950 4350 50  0001 C CNN
+	1    5950 4350
+	1    0    0    -1
+$EndComp
+Wire Wire Line
+	5950 4100 5950 4350
+Text GLabel 6300 2450 0    50   Input ~ 0
+Vbat
+Wire Wire Line
+	6300 2450 6500 2450
+Text GLabel 2450 1450 2    50   Input ~ 0
+Vbat
+Wire Wire Line
+	2450 1450 2050 1450
+Wire Wire Line
+	2050 1450 2050 1650
 $EndSCHEMATC
