File: kicad/eboard.kicad_pcb (KiCad board)
At the start: 2 copper layers, 42 parts, among them J1 Conn_01x02_Male, J2 USB_B_Micro, J3 Conn_01x03_Male, J4 Conn_01x02_Male, J5 Conn_01x02_Male, Q1 AO4407A, U1 ESP32-PICO-D4, U2 TPS63000, U3 TP4056, U4 SRV05-4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

Commit message: wip
Parts:
- removed C8: 100n, Capacitor_SMD:C_0402_1005Metric
- moved C1 137.9 mm to (50.1, 38.6), turned to 180 degrees
- moved C4 137.4 mm to (50.1, 42.5), turned to 180 degrees
- moved C2 136.6 mm to (50.1, 41.3), turned to 180 degrees
- moved C6 133.5 mm to (50.1, 40.1), turned to 180 degrees
- moved C5 129.3 mm to (54.2, 37.1), turned to 90 degrees
- moved C3 127.8 mm to (58.7, 37.3), turned to 90 degrees
- moved C7 125.6 mm to (56.2, 48.3), turned to 270 degrees
- moved C16 112.5 mm to (64.5, 47.2), turned to 180 degrees
- moved C9 103.8 mm to (87.1, 41.6), turned to 270 degrees
- moved D3 103.0 mm to (67.4, 69.0)
- moved C10 96.9 mm to (88.7, 47.8)
- moved FB2 96.7 mm to (67.4, 72.8), turned to 180 degrees
- moved C12 96.2 mm to (94.1, 44.2), turned to 180 degrees
- moved R7 94.4 mm to (90.9, 46.1), turned to 180 degrees
- moved U2 93.2 mm to (90.1, 42.3), turned to 270 degrees
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Connections:
- U3 pad 9: (no net) -> GND
- U4 pad 3: USB_DM -> (no net)
- U4 pad 6: (no net) -> USB_DM
Routing:
- net Net-(C11-Pad1): track 0.00 -> 41.0 mm
- net Vraw: track 0.00 -> 34.8 mm
- net GND: track 0.00 -> 26.4 mm
- net +3V3: track 0.00 -> 24.3 mm
- net PSRAM_CS: track 0.00 -> 13.8 mm, vias 0 -> 2
- net SIO2: track 0.00 -> 13.3 mm
- net SIO1: track 0.00 -> 13.3 mm
- net VDD_SDIO: track 0.00 -> 8.26 mm
- net Net-(C12-Pad2): track 0.00 -> 6.42 mm
- net SIO3: track 0.00 -> 6.24 mm
- net SCLK: track 0.00 -> 5.93 mm
- net SIO0: track 0.00 -> 5.89 mm
- net Net-(D1-Pad1): track 0.00 -> 4.21 mm
- net Net-(L1-Pad2): track 0.00 -> 4.19 mm
- net Net-(D2-Pad1): track 0.00 -> 4.13 mm
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Other:
- board outline added: 90 x 90 mm
- copper layers 2 -> 4
