File: kicad/eboard.sch (KiCad schematic (older format))
At the start: 14 parts

Commit message: dcdc
Parts:
- added C? (x2): 10u, Capacitor_SMD:C_0402_1005Metric, symbol pace:10u
- added D?: SS210, Diode_SMD:D_SMA, symbol pace:SS210
- added F? (x2): fuse, Fuse:Fuse_0805_2012Metric, symbol pace:fuse
- added FB? (x2): bead, Inductor_SMD:L_0805_2012Metric, symbol pace:bead
- added J?: Conn_01x02_Male, symbol Connector:Conn_01x02_Male
- added Q? (x2): AO4407A, Package_SO:SOIC-8_3.9x4.9mm_P1.27mm, symbol pace:AO4407A
- added R?: 100, Resistor_SMD:R_0402_1005Metric, symbol pace:100
- added R? (x3): 100k, Resistor_SMD:R_0402_1005Metric, symbol pace:100k
- added SW?: SWITCH, symbol switch_spdt:SWITCH
- added U?: AP1117-33, Package_TO_SOT_SMD:SOT-223-3_TabPin2, symbol pace:AP1117-33
Connections:
- net labels added: USB_DM, USB_DP, Vdc, Vusb
- wire segments 20 -> 68
- no-connect marks 1 -> 3
Other:
- note added: "2v to 5.5v"
- note added: "7v absolute max\n"
- note added: "Change to TPS63001\n"
- note added: "Reverse polarity protection"
- note added: "Switch between usb and battery"
- moved on the sheet: J?, U?

Commit message: lib
Parts:
- SW?: symbol switch_spdt:SWITCH -> eboard-rescue:SWITCH-switch_spdt
Changed lines of the file:
@@
 Connection ~ 7000 1250
 $Comp
-L switch_spdt:SWITCH SW?
+L eboard-rescue:SWITCH-switch_spdt SW?
 U 1 1 5FA509A0
 P 9050 2600

Commit message: power
Parts:
- removed C? (x2): 10u, Capacitor_SMD:C_0402_1005Metric, symbol pace:10u
- removed D?: SS210, Diode_SMD:D_SMA, symbol pace:SS210
- removed Q? (x2): AO4407A, Package_SO:SOIC-8_3.9x4.9mm_P1.27mm, symbol pace:AO4407A
- removed R?: 100, Resistor_SMD:R_0402_1005Metric, symbol pace:100
- removed R? (x3): 100k, Resistor_SMD:R_0402_1005Metric, symbol pace:100k
- removed SW?: SWITCH, symbol eboard-rescue:SWITCH-switch_spdt
- removed U?: AP1117-33, Package_TO_SOT_SMD:SOT-223-3_TabPin2, symbol pace:AP1117-33
- added C? (x2): 10u, Capacitor_SMD:C_0402_1005Metric, symbol pace:10u
- added D? (x2): ledred, LED_SMD:LED_0603_1608Metric, symbol pace:ledred
- added D?: SS210, Diode_SMD:D_SMA, symbol pace:SS210
- added J? (x2): Conn_01x02_Male, symbol Connector:Conn_01x02_Male
- added J?: Conn_01x03_Male, symbol Connector:Conn_01x03_Male
- added Q?: AO4407A, Package_SO:SOIC-8_3.9x4.9mm_P1.27mm, symbol pace:AO4407A
- added R? (x3): 10k, Resistor_SMD:R_0402_1005Metric, symbol pace:10k
- added U?: TP4056, symbol pace:TP4056
Connections:
- net labels added: Vin, Vraw
- net labels removed: Vdc, Vusb
- wire segments 68 -> 77
Other:
- note removed: "Change to TPS63001\n"
- note removed: "Reverse polarity protection"
- note removed: "Switch between usb and battery"
- moved on the sheet: C?, F?, FB?, J?, U?

Commit message: power
Parts:
- removed D? (x2): ledred, LED_SMD:LED_0603_1608Metric, symbol pace:ledred
- removed F? (x2): fuse, Fuse:Fuse_0805_2012Metric, symbol pace:fuse
- removed R?: 10k, Resistor_SMD:R_0402_1005Metric, symbol pace:10k
- removed U?: TP4056, symbol pace:TP4056
- added C10: 100n, Capacitor_SMD:C_0402_1005Metric, symbol pace:100n
- added C12: 2.2pF, Capacitor_SMD:C_0402_1005Metric, symbol pace:2.2pF
- added C14, C15, C9: 10u, Capacitor_SMD:C_0402_1005Metric, symbol pace:10u
- added D1: ledgreen, LED_SMD:LED_0603_1608Metric, symbol pace:ledgreen
- added D2: ledyellow, LED_SMD:LED_0603_1608Metric, symbol pace:ledyellow
- added L1: 2.2uH, Inductor_SMD:L_Coilcraft_XxL4020, symbol pace:2.2uH
- added R1, R6: 1meg, Resistor_SMD:R_0603_1608Metric, symbol pace:1meg
- added R3, R4: 10k, Resistor_SMD:R_0402_1005Metric, symbol pace:10k
- added R5: 100, Resistor_SMD:R_0402_1005Metric, symbol pace:100
- added R7: 180k, Resistor_SMD:R_0603_1608Metric, symbol pace:180k
- added U2: TPS63000, Package_SON:Texas_DRC0010J_ThermalVias, symbol pace:TPS63000
- added U3: TP4056, Package_SO:SOIC-8-1EP_3.9x4.9mm_P1.27mm_EP2.29x3mm_ThermalVias, symbol pace:TP4056
- J1, J4, J5: renamed from J?; footprint (none) -> Connector_PinHeader_2.54mm:PinHeader_1x02_P2.54mm_Vertical
- J3: renamed from J?; footprint (none) -> Connector_PinHeader_2.54mm:PinHeader_1x03_P2.54mm_Vertical
- gave numbers to parts that had none: 22
Connections:
- net +3V3: now also C12.1, C14.1, C15.1, R6.1, U2.1 (VOUT)
- net GND: now also C10.2, C14.2, C15.2, C9.2, R1.2, R7.2, U2.11 (PGND), U2.3 (PGND), U2.9 (GND), U3.1 (TEMP), U3.3 (GND)
- net Vin: now also C9.1, U2.5 (VIN)
- net Vraw: now also U3.5 (BAT)
- net at J1.1 (Pin_1): now also FB1.2
- net at J2.1 (VBUS), U4.5 (VP): now also FB2.2
- net at R2.1: now also D1.2 (A)
- net at C11.1, J3.1 (Pin_1), R2.2: now also R1.1, R3.1, R4.1, U3.4 (VCC), U3.8 (CE)
- net at R8.1: now also U3.2 (PROG)
- new net: C12.2, R6.2, R7.1, U2.10 (FB)
- new net: L1.2, U2.2 (L2)
- new net: L1.1, U2.4 (L1)
- new net: R5.1, U2.6 (EN), U2.7 (PS/SYNC), U2.8 (VINA)
- new net: D1.1 (K), U3.6 (~STDBY)
- new net: D2.1 (K), U3.7 (~CHRG)
- new net: C10.1, R5.2
- new net: D2.2 (A), R3.2, R4.2
Other:
- note added: "1.8 to 4.6 volts"
- note added: "3.28v nominal\nwith 1% reisistors: 3.00 to 3.33v"
- note added: "Connect 1-2: lithium battery with recharge\nConnect 2-3: external DC supply"
- note added: "Connect single Li-ion or LiPo\nto one of these connectors"
- note added: "Diode drops 5v usb input\nto safe range for dc-dc converter"
- note added: "ESD protection"
- note added: "Includes short circuit\nprotection"
- note added: "Lithium battery charger"
- note added: "Reverse polarity\nprotection"
- note added: "dc-dc converter / regulator"
- note removed: "2v to 5.5v"
- note removed: "7v absolute max\n"
- moved on the sheet: C1, C11, C13, C2, C3, C4, C5, C6, C7, C8, D3, FB1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

Commit message: wip
Parts:
- removed C8: 100n, Capacitor_SMD:C_0402_1005Metric, symbol pace:100n
Connections:
- net GND: now also U3.9 (PAD)
- net USB_DM: now also U4.6 (IO4); no longer U4.3 (IO2)
Other:
- moved on the sheet: D3, FB2, R8, U4
Changed lines of the file:
@@
 L pace:SRV05-4 U4
 U 1 1 5FA85788
-P 4200 1400
-F 0 "U4" H 4450 900 50  0000 C CNN
-F 1 "SRV05-4" H 4600 800 50  0000 C CNN
-F 2 "Package_TO_SOT_SMD:SOT-23-6" H 4900 950 50  0001 C CNN
-F 3 "http://www.onsemi.com/pub/Collateral/SRV05-4-D.PDF" H 4200 1400 50  0001 C CNN
-F 4 "C85364" H 4200 1400 50  0001 C CNN "LCSC"
-	1    4200 1400
+P 4500 1400
+F 0 "U4" H 4750 900 50  0000 C CNN
+F 1 "SRV05-4" H 4900 800 50  0000 C CNN
+F 2 "Package_TO_SOT_SMD:SOT-23-6" H 5200 950 50  0001 C CNN
+F 3 "http://www.onsemi.com/pub/Collateral/SRV05-4-D.PDF" H 4500 1400 50  0001 C CNN
+F 4 "C85364" H 4500 1400 50  0001 C CNN "LCSC"
+	1    4500 1400
 	1    0    0    -1
 $EndComp
@@
 L power:GND #PWR?
 U 1 1 5F9FE0F5
-P 4200 1900
-F 0 "#PWR?" H 4200 1650 50  0001 C CNN
-F 1 "GND" H 4205 1727 50  0000 C CNN
-F 2 "" H 4200 1900 50  0001 C CNN
-F 3 "" H 4200 1900 50  0001 C CNN
-	1    4200 1900
+P 4500 1900
+F 0 "#PWR?" H 4500 1650 50  0001 C CNN
+F 1 "GND" H 4505 1727 50  0000 C CNN
+F 2 "" H 4500 1900 50  0001 C CNN
+F 3 "" H 4500 1900 50  0001 C CNN
+	1    4500 1900
 	1    0    0    -1
 $EndComp
@@
 NoConn ~ 3100 1500
 Wire Wire Line
-	3100 1300 3250 1300
-Wire Wire Line
-	3100 1400 3250 1400
-Wire Wire Line
-	3450 1400 3450 1500
-Wire Wire Line
-	3450 1500 3700 1500
-Text GLabel 3300 1150 2    50   Input ~ 0
+	3100 1300 3150 1300
+Wire Wire Line
+	3100 1400 3150 1400
+Text GLabel 3150 1300 2    50   Input ~ 0
 USB_DP
-Wire Wire Line
-	3300 1150 3250 1150
-Wire Wire Line
-	3250 1150 3250 1300
-Connection ~ 3250 1300
-Wire Wire Line
-	3250 1300 3700 1300
-Text GLabel 3300 1750 2    50   Input ~ 0
+Text GLabel 3150 1400 2    50   Input ~ 0
 USB_DM
-Wire Wire Line
-	3300 1750 3250 1750
-Wire Wire Line
-	3250 1750 3250 1400
-Connection ~ 3250 1400
-Wire Wire Line
-	3250 1400 3450 1400
-Text GLabel 5000 700  2    50   Input ~ 0
+Text GLabel 5250 700  2    50   Input ~ 0
 Vin
 Wire Wire Line
@@
 L pace:bead FB2
 U 1 1 5FA2A41A
-P 4500 700
-F 0 "FB2" V 4355 700 50  0000 C CNN
-F 1 "bead" V 4354 700 50  0001 C CNN
-F 2 "Inductor_SMD:L_0805_2012Metric" V 4430 700 50  0001 C CNN
-F 3 "https://datasheet.lcsc.com/szlcsc/Sunlord-GZ2012D101TF_C1015.pdf" H 4500 700 50  0001 C CNN
-F 4 "C1015" H 4500 700 50  0001 C CNN "LCSC"
-	1    4500 700
+P 4750 700
+F 0 "FB2" V 4605 700 50  0000 C CNN
+F 1 "bead" V 4604 700 50  0001 C CNN
+F 2 "Inductor_SMD:L_0805_2012Metric" V 4680 700 50  0001 C CNN
+F 3 "https://datasheet.lcsc.com/szlcsc/Sunlord-GZ2012D101TF_C1015.pdf" H 4750 700 50  0001 C CNN
+F 4 "C1015" H 4750 700 50  0001 C CNN "LCSC"
+	1    4750 700
 	0    1    1    0
 $EndComp
@@
 $EndComp
 Wire Wire Line
-	3200 700  4200 700
-Wire Wire Line
-	4200 700  4200 900
+	3200 700  4500 700
+Wire Wire Line
+	4500 700  4500 900
 Wire Wire Line
 	3200 700  3200 1100
@@
 L pace:SS210 D3
 U 1 1 5FACDF9F
-P 4750 700
-F 0 "D3" H 4750 493 50  0000 C CNN
-F 1 "SS210" H 4750 584 50  0000 C CNN
-F 2 "Diode_SMD:D_SMA" V 4750 700 50  0001 C CNN
-F 3 "https://datasheet.lcsc.com/szlcsc/1903041730_MDD-Jiangsu-Yutai-Elec-SS210_C14996.pdf" V 4750 700 50  0001 C CNN
-F 4 "C14996" H 4750 700 50  0001 C CNN "LCSC"
-	1    4750 700
+P 5000 700
+F 0 "D3" H 5000 493 50  0000 C CNN
+F 1 "SS210" H 5000 584 50  0000 C CNN
+F 2 "Diode_SMD:D_SMA" V 5000 700 50  0001 C CNN
+F 3 "https://datasheet.lcsc.com/szlcsc/1903041730_MDD-Jiangsu-Yutai-Elec-SS210_C14996.pdf" V 5000 700 50  0001 C CNN
+F 4 "C14996" H 5000 700 50  0001 C CNN "LCSC"
+	1    5000 700
 	-1   0    0    1
 $EndComp
 Wire Wire Line
-	4600 700  4650 700
-Wire Wire Line
-	4850 700  5000 700
+	4850 700  4900 700
+Wire Wire Line
+	5100 700  5250 700
 $Comp
 L pace:AO4407A Q1
@@
 L pace:10k R8
 U 1 1 5FAB7004
-P 3300 3600
-F 0 "R8" H 3359 3646 50  0000 L CNN
-F 1 "10k" H 3359 3555 50  0000 L CNN
-F 2 "Resistor_SMD:R_0402_1005Metric" H 3300 3600 50  0001 C CNN
-F 3 "https://datasheet.lcsc.com/szlcsc/Uniroyal-Elec-0402WGF1002TCE_C25744.pdf" H 3300 3600 50  0001 C CNN
-F 4 "C25744" H 3300 3600 50  0001 C CNN "LCSC"
-	1    3300 3600
-	1    0    0    -1
-$EndComp
-Wire Wire Line
-	3250 3350 3300 3350
-Wire Wire Line
-	3300 3350 3300 3500
-$Comp
-L power:GND #PWR?
-U 1 1 5FABCA2F
-P 3300 3700
-F 0 "#PWR?" H 3300 3450 50  0001 C CNN
-F 1 "GND" H 3305 3527 50  0000 C CNN
-F 2 "" H 3300 3700 50  0001 C CNN
-F 3 "" H 3300 3700 50  0001 C CNN
-	1    3300 3700
-	1    0    0    -1
-$EndComp
+P 3400 3600
+F 0 "R8" H 3459 3646 50  0000 L CNN
+F 1 "10k" H 3459 3555 50  0000 L CNN
+F 2 "Resistor_SMD:R_0402_1005Metric" H 3400 3600 50  0001 C CNN
+F 3 "https://datasheet.lcsc.com/szlcsc/Uniroyal-Elec-0402WGF1002TCE_C25744.pdf" H 3400 3600 50  0001 C CNN
+F 4 "C25744" H 3400 3600 50  0001 C CNN "LCSC"
+	1    3400 3600
+	1    0    0    -1
+$EndComp
+Wire Wire Line
+	3250 3350 3400 3350
+Wire Wire Line
+	3400 3350 3400 3500
 $Comp
 L power:GND #PWR?
 U 1 1 5FABF7F3
-P 3550 3700
-F 0 "#PWR?" H 3550 3450 50  0001 C CNN
-F 1 "GND" H 3555 3527 50  0000 C CNN
-F 2 "" H 3550 3700 50  0001 C CNN
-F 3 "" H 3550 3700 50  0001 C CNN
-	1    3550 3700
-	1    0    0    -1
-$EndComp
-Wire Wire Line
-	3250 3250 3550 3250
-Wire Wire Line
-	3550 3250 3550 3700
+P 3600 3700
+F 0 "#PWR?" H 3600 3450 50  0001 C CNN
+F 1 "GND" H 3605 3527 50  0000 C CNN
+F 2 "" H 3600 3700 50  0001 C CNN
+F 3 "" H 3600 3700 50  0001 C CNN
+	1    3600 3700
+	1    0    0    -1
+$EndComp
+Wire Wire Line
+	3250 3250 3600 3250
+Wire Wire Line
+	3600 3250 3600 3700
 $Comp
 L pace:10u C11
@@
 Wire Wire Line
 	2050 3050 1700 3050
-$Comp
-L pace:TPS63000 U2
-U 1 1 5FA83D18
-P 2450 5250
-F 0 "U2" H 2450 5917 50  0000 C CNN
-F 1 "TPS63000" H 2450 5826 50  0000 C CNN
-F 2 "Package_SON:Texas_DRC0010J_ThermalVias" H 3300 4700 50  0001 C CNN
-F 3 "http://www.ti.com/lit/ds/symlink/tps63000.pdf" H 2150 5800 50  0001 C CNN
-	1    2450 5250
-	1    0    0    -1
-$EndComp
 $Comp
 L pace:2.2uH L1
@@
 $EndComp
 Wire Wire Line
-	4400 700  4200 700
-Connection ~ 4200 700
+	4650 700  4500 700
+Connection ~ 4500 700
 Text Notes 4000 3800 0    50   ~ 0
 Connect single Li-ion or LiPo\nto one of these connectors
@@
 	8750 2200 8850 2200
 Wire Wire Line
-	9650 1000 10000 1000
-Connection ~ 9650 1000
-Wire Wire Line
 	9250 1000 9650 1000
 Connection ~ 9250 1000
@@
 Wire Wire Line
 	7200 1000 7650 1000
-Wire Wire Line
-	9650 800  10000 800
-Connection ~ 9650 800
 Wire Wire Line
 	9250 800  9650 800
@@
 $EndComp
 $Comp
-L pace:100n C8
-U 1 1 5FA00E4A
-P 10000 900
-F 0 "C8" H 10092 946 50  0000 L CNN
-F 1 "100n" H 10092 855 50  0000 L CNN
-F 2 "Capacitor_SMD:C_0402_1005Metric" H 10000 900 50  0001 C CNN
-F 3 "https://datasheet.lcsc.com/szlcsc/Samsung-Electro-Mechanics-CL05B104KO5NNNC_C1525.pdf" H 10000 900 50  0001 C CNN
-F 4 "C1525" H 10000 900 50  0001 C CNN "LCSC"
-	1    10000 900
-	1    0    0    -1
-$EndComp
-$Comp
 L pace:100n C7
 U 1 1 5FA00097
@@
 	1    0    0    -1
 $EndComp
+$Comp
+L power:GND #PWR?
+U 1 1 5FABCA2F
+P 3400 3700
+F 0 "#PWR?" H 3400 3450 50  0001 C CNN
+F 1 "GND" H 3405 3527 50  0000 C CNN
+F 2 "" H 3400 3700 50  0001 C CNN
+F 3 "" H 3400 3700 50  0001 C CNN
+	1    3400 3700
+	1    0    0    -1
+$EndComp
+$Comp
+L power:GND #PWR?
+U 1 1 5FAC67E2
+P 3250 3700
+F 0 "#PWR?" H 3250 3450 50  0001 C CNN
+F 1 "GND" H 3255 3527 50  0000 C CNN
+F 2 "" H 3250 3700 50  0001 C CNN
+F 3 "" H 3250 3700 50  0001 C CNN
+	1    3250 3700
+	1    0    0    -1
+$EndComp
+Wire Wire Line
+	3250 3450 3250 3700
+Text GLabel 5000 1500 2    50   Input ~ 0
+USB_DM
+Text GLabel 4000 1300 0    50   Input ~ 0
+USB_DP
+$Comp
+L pace:TPS63000 U2
+U 1 1 5FB2B195
+P 2450 5250
+F 0 "U2" H 2450 5917 50  0000 C CNN
+F 1 "TPS63000" H 2450 5826 50  0000 C CNN
+F 2 "Package_SON:Texas_DRC0010J_ThermalVias" H 3300 4700 50  0001 C CNN
+F 3 "http://www.ti.com/lit/ds/symlink/tps63000.pdf" H 2150 5800 50  0001 C CNN
+	1    2450 5250
+	1    0    0    -1
+$EndComp
