File: eboard/eboard.kicad_pcb (KiCad board)
At the start: 4 copper layers, 90 x 90 mm, 41 parts, among them J1 Conn_01x02_Male, J2 USB_B_Micro, J3 Conn_01x03_Male, J4 Conn_01x02_Male, J5 Conn_01x02_Male, Q1 AO4407A, U1 ESP32-PICO-D4, U2 TPS63000, U3 TP4056, U4 SRV05-4, U5 CP2102, U6 W25Q128JVSIQ

Commit message: routing
Parts:
- added AE1: Antenna_Shield, Connector_Coaxial:SMA_Samtec_SMA-J-P-X-ST-EM1_EdgeMount, F.Cu at (41.8, 46.4)
- added C17: 2.2pF, Capacitor_SMD:C_0402_1005Metric, F.Cu at (95.4, 68.6)
- added C18: 10u, Capacitor_SMD:C_0402_1005Metric, F.Cu at (93.3, 70.6)
- added C19: 10u, Capacitor_SMD:C_0402_1005Metric, F.Cu at (93.4, 69.1)
- added C20: 100n, Capacitor_SMD:C_0402_1005Metric, F.Cu at (48.0, 58.4)
- added C21: 100n, Capacitor_SMD:C_0402_1005Metric, F.Cu at (96.0, 42.9)
- added C22: 330pF, Capacitor_SMD:C_0402_1005Metric, F.Cu at (51.3, 48.3)
- added C23: 1u, Capacitor_SMD:C_0402_1005Metric, F.Cu at (96.0, 41.9)
- added C24: 330pF, Capacitor_SMD:C_0402_1005Metric, F.Cu at (50.8, 49.8)
- added C8: 10u, Capacitor_SMD:C_0402_1005Metric, F.Cu at (93.1, 76.7)
- added D4: ledgreen, LED_SMD:LED_0603_1608Metric, F.Cu at (64.2, 44.0)
- added D5: SS210, Diode_SMD:D_SMA, F.Cu at (104.1, 91.4)
- added H1: MountingHole, MountingHole:MountingHole_3.2mm_M3, F.Cu at (43.4, 116.6)
- added H2: MountingHole, MountingHole:MountingHole_3.2mm_M3, F.Cu at (43.2, 33.5)
- added H3: MountingHole, MountingHole:MountingHole_3.2mm_M3, F.Cu at (126.5, 33.5)
- added H4: MountingHole, MountingHole:MountingHole_3.2mm_M3, F.Cu at (126.5, 116.3)
- added J10: Conn_01x06_Male, Connector_PinHeader_2.54mm:PinHeader_1x06_P2.54mm_Vertical, F.Cu at (101.6, 111.8)
- added J11: Conn_01x02_Male, Connector_PinHeader_2.54mm:PinHeader_1x02_P2.54mm_Vertical, F.Cu at (46.8, 43.1)
- added J12: Conn_01x02_Male, Connector_PinHeader_2.54mm:PinHeader_1x02_P2.54mm_Vertical, F.Cu at (44.7, 86.1)
- added J13: Conn_01x02_Male, Connector_PinHeader_2.54mm:PinHeader_1x02_P2.54mm_Vertical, F.Cu at (44.7, 93.7)
- added J14: Conn_01x02_Male, Connector_PinHeader_2.54mm:PinHeader_1x02_P2.54mm_Vertical, F.Cu at (44.7, 101.3)
- added J15: Conn_01x02_Male, Connector_PinHeader_2.54mm:PinHeader_1x02_P2.54mm_Vertical, F.Cu at (44.7, 109.0)
- added J16: Conn_01x03_Male, Connector_PinHeader_2.54mm:PinHeader_1x03_P2.54mm_Vertical, F.Cu at (86.4, 111.8)
- added J17: Conn_01x03_Male, Connector_PinHeader_2.54mm:PinHeader_1x03_P2.54mm_Vertical, F.Cu at (76.2, 111.8)
- added J18: Conn_01x03_Male, Connector_PinHeader_2.54mm:PinHeader_1x03_P2.54mm_Vertical, F.Cu at (81.3, 111.8)
- added J19: Conn_01x03_Male, Connector_PinHeader_2.54mm:PinHeader_1x03_P2.54mm_Vertical, F.Cu at (71.1, 111.8)
- added J20: Conn_01x02_Male, Connector_PinHeader_2.54mm:PinHeader_1x02_P2.54mm_Vertical, F.Cu at (44.7, 78.5)
- added J21: Conn_01x03_Male, Connector_PinHeader_2.54mm:PinHeader_1x03_P2.54mm_Vertical, F.Cu at (49.8, 78.5)
- added J6: Conn_01x03_Male, Connector_PinHeader_2.54mm:PinHeader_1x03_P2.54mm_Vertical, F.Cu at (104.9, 53.6)
- added J7: Conn_01x04_Male, Connector_PinHeader_2.54mm:PinHeader_1x04_P2.54mm_Vertical, F.Cu at (96.5, 111.8)
- added J8: Conn_01x04_Male, Connector_PinHeader_2.54mm:PinHeader_1x04_P2.54mm_Vertical, F.Cu at (91.4, 111.8)
- added J9: Conn_01x06_Male, Connector_PinHeader_2.54mm:PinHeader_1x06_P2.54mm_Vertical, F.Cu at (106.7, 111.8)
- added L2: 2.2uH, Inductor_SMD:L_Coilcraft_XxL4020, F.Cu at (88.2, 73.4)
- added Q10: BSS138K, Package_TO_SOT_SMD:SOT-23, F.Cu at (57.5, 106.4)
- added Q11: AO4407A_new, Package_SO:SOIC-8_3.9x4.9mm_P1.27mm, F.Cu at (51.3, 107.6)
- added Q12: BSS138K, Package_TO_SOT_SMD:SOT-23, F.Cu at (61.4, 84.2)
- added Q13: BSS138K, Package_TO_SOT_SMD:SOT-23, F.Cu at (61.4, 91.2)
- added Q14: BSS138K, Package_TO_SOT_SMD:SOT-23, F.Cu at (61.5, 99.2)
- added Q15: BSS138K, Package_TO_SOT_SMD:SOT-23, F.Cu at (57.5, 84.1)
- added Q16: BSS138K, Package_TO_SOT_SMD:SOT-23, F.Cu at (57.4, 91.3)
- added Q17: BSS138K, Package_TO_SOT_SMD:SOT-23, F.Cu at (57.4, 99.2)
- added Q18: AO4407A_new, Package_SO:SOIC-8_3.9x4.9mm_P1.27mm, F.Cu at (51.3, 85.1)
- added Q19: AO4407A_new, Package_SO:SOIC-8_3.9x4.9mm_P1.27mm, F.Cu at (51.3, 92.2)
- added Q2: S8050, Package_TO_SOT_SMD:SOT-23, F.Cu at (66.0, 49.0)
- added Q20: AO4407A_new, Package_SO:SOIC-8_3.9x4.9mm_P1.27mm, F.Cu at (51.3, 100.2)
- added Q3: S8050, Package_TO_SOT_SMD:SOT-23, F.Cu at (66.0, 53.3)
- added Q4: BSS138K, Package_TO_SOT_SMD:SOT-23, F.Cu at (86.5, 97.9)
- added Q5: BSS138K, Package_TO_SOT_SMD:SOT-23, F.Cu at (86.2, 92.1)
- added Q6: AO4407A_new, Package_SO:SOIC-8_3.9x4.9mm_P1.27mm, F.Cu at (103.5, 76.2)
- added Q7: BSS138K, Package_TO_SOT_SMD:SOT-23, F.Cu at (75.7, 58.1)
- added Q8: BSS138K, Package_TO_SOT_SMD:SOT-23, F.Cu at (80.4, 58.2)
- added Q9: BSS138K, Package_TO_SOT_SMD:SOT-23, F.Cu at (61.7, 106.5)
- added R10: 1meg, Resistor_SMD:R_0603_1608Metric, F.Cu at (98.9, 65.7)
- added R11: 100k, Resistor_SMD:R_0402_1005Metric, F.Cu at (98.5, 71.8)
- added R12: 100k, Resistor_SMD:R_0402_1005Metric, F.Cu at (48.3, 54.1)
- added R13: 100k, Resistor_SMD:R_0402_1005Metric, F.Cu at (50.3, 54.1)
- added R14: 100k, Resistor_SMD:R_0402_1005Metric, F.Cu at (48.3, 55.6)
- added R15: 10k, Resistor_SMD:R_0402_1005Metric, F.Cu at (95.4, 48.1)
- added R16: 10k, Resistor_SMD:R_0402_1005Metric, F.Cu at (64.3, 42.0)
- added R17: 10k, Resistor_SMD:R_0402_1005Metric, F.Cu at (68.8, 49.8)
- added R18: 10k, Resistor_SMD:R_0402_1005Metric, F.Cu at (68.8, 53.6)
- added R19: 10k, Resistor_SMD:R_0402_1005Metric, F.Cu at (48.0, 57.1)
- added R20: 10k, Resistor_SMD:R_0402_1005Metric, F.Cu at (62.0, 56.1)
- added R21: 3.3k, Resistor_SMD:R_0402_1005Metric, F.Cu at (89.9, 99.2)
- added R22: 3.3k, Resistor_SMD:R_0402_1005Metric, F.Cu at (89.5, 92.4)
- added R23: 3.3k, Resistor_SMD:R_0402_1005Metric, F.Cu at (83.4, 98.5)
- added R24: 3.3k, Resistor_SMD:R_0402_1005Metric, F.Cu at (83.1, 92.9)
- added R25: 3.3k, Resistor_SMD:R_0402_1005Metric, F.Cu at (104.1, 88.9)
- added R26: 10k, Resistor_SMD:R_0402_1005Metric, F.Cu at (98.6, 68.7)
- added R27: 100, Resistor_SMD:R_0402_1005Metric, F.Cu at (101.9, 70.9)
- added R28: 100, Resistor_SMD:R_0402_1005Metric, F.Cu at (72.7, 59.0)
- added R29: 100k, Resistor_SMD:R_0402_1005Metric, F.Cu at (72.7, 56.7)
- added R30: 100, Resistor_SMD:R_0402_1005Metric, F.Cu at (62.4, 109.4)
- added R31: 100k, Resistor_SMD:R_0402_1005Metric, F.Cu at (59.3, 109.4)
- added R32: 100k, Resistor_SMD:R_0402_1005Metric, F.Cu at (56.9, 109.4)
- added R33: 100, Resistor_SMD:R_0402_1005Metric, F.Cu at (62.1, 87.0)
- added R34: 100, Resistor_SMD:R_0402_1005Metric, F.Cu at (62.1, 94.2)
- added R35: 100, Resistor_SMD:R_0402_1005Metric, F.Cu at (62.3, 102.1)
- added R36: 100k, Resistor_SMD:R_0402_1005Metric, F.Cu at (58.9, 87.0)
- added R37: 100k, Resistor_SMD:R_0402_1005Metric, F.Cu at (58.9, 94.1)
- added R38: 100k, Resistor_SMD:R_0402_1005Metric, F.Cu at (58.9, 102.0)
- added R39: 100k, Resistor_SMD:R_0402_1005Metric, F.Cu at (56.6, 87.0)
- added R40: 100k, Resistor_SMD:R_0402_1005Metric, F.Cu at (56.6, 94.1)
- added R41: 100k, Resistor_SMD:R_0402_1005Metric, F.Cu at (56.3, 102.0)
- added R42: 100k, Resistor_SMD:R_0402_1005Metric, F.Cu at (50.3, 55.6)
- added R9: 100, Resistor_SMD:R_0402_1005Metric, F.Cu at (96.8, 76.3)
- added SW1: pushbutton_switch, Button_Switch_THT:SW_PUSH_6mm, F.Cu at (45.5, 67.1)
- added SW2: pushbutton_switch, Button_Switch_THT:SW_PUSH_6mm, F.Cu at (57.1, 67.1)
- added U7: SRV05-4, Package_TO_SOT_SMD:SOT-23-6, F.Cu at (95.4, 99.2)
- added U8: SRV05-4, Package_TO_SOT_SMD:SOT-23-6, F.Cu at (103.9, 95.5)
- added U9: SRV05-4, Package_TO_SOT_SMD:SOT-23-6, F.Cu at (78.7, 101.6)
- J4: value Conn_01x02_Male -> jst_battery; footprint Connector_PinHeader_2.54mm:PinHeader_1x02_P2.54mm_Vertical -> Connector_JST:JST_PH_B2B-PH-K_1x02_P2.00mm_Vertical
- Q1: value AO4407A -> AO4407A_new
- R1: value 1meg -> 100k; footprint Resistor_SMD:R_0603_1608Metric -> Resistor_SMD:R_0402_1005Metric
- U6: value W25Q128JVSIQ -> TPS63000; footprint Package_SO:SOIC-8_5.23x5.23mm_P1.27mm -> Package_SON:Texas_DRC0010J_ThermalVias
- moved J1 70.0 mm to (109.2, 33.0), turned to 90 degrees
- moved J2 68.4 mm to (99.1, 33.3), turned to 180 degrees
- moved FB1 65.9 mm to (110.7, 36.4)
- moved Q1 58.6 mm to (110.8, 41.3), turned to 0 degrees
- moved U4 58.5 mm to (99.1, 39.1), turned to 0 degrees
- moved FB2 49.9 mm to (103.3, 38.1), turned to 90 degrees
- moved R2 48.9 mm to (74.7, 53.3), turned to 270 degrees
- moved R3 47.3 mm to (78.7, 53.6), turned to 90 degrees
- moved J4 47.0 mm to (76.2, 33.0)
- moved D3 45.1 mm to (104.9, 43.9), turned to 90 degrees
- moved C16 44.8 mm to (99.1, 75.7), turned to 90 degrees
- moved R4 44.8 mm to (79.9, 53.5), turned to 90 degrees
- moved U5 44.5 mm to (99.3, 45.6), turned to 270 degrees
- moved D1 44.4 mm to (76.7, 53.6), turned to 90 degrees
- moved D2 41.0 mm to (81.4, 53.9), turned to 90 degrees
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Connections:
- net Net-(C11-Pad1) renamed Vcharge
- C12 pad 1: +3V3 -> Net-(C12-Pad1)
- C16 pad 1: VDD_SDIO -> Net-(C16-Pad1)
- C9 pad 1: Vin -> Vraw
- R6 pad 1: +3V3 -> Net-(C12-Pad1)
- U1 pad 10: (no net) -> ADC0
- U1 pad 11: (no net) -> ADC1
- U1 pad 13: (no net) -> OUT3
- U1 pad 14: (no net) -> OUT2
- U1 pad 15: (no net) -> IO3
- U1 pad 16: (no net) -> OUT1
- U1 pad 17: (no net) -> OUT0
- U1 pad 18: (no net) -> IO2
- U1 pad 2: (no net) -> WIFI
- U1 pad 20: (no net) -> IO1
- U1 pad 21: (no net) -> SPI_CS0
- U1 pad 22: (no net) -> DISABLE_5v
- U1 pad 23: (no net) -> BOOT0
- U1 pad 24: (no net) -> IO0
- U1 pad 26: VDD_SDIO -> (no net)
- U1 pad 27: SIO1 -> (no net)
- U1 pad 28: (no net) -> ENABLE_STATUS
- U1 pad 29: PSRAM_CS -> SPI_CS1
- U1 pad 30: SIO3 -> (no net)
- U1 pad 31: SCLK -> (no net)
- U1 pad 32: SIO2 -> (no net)
- U1 pad 33: SIO0 -> (no net)
- U1 pad 34: (no net) -> STATUS_LED
- U1 pad 35: (no net) -> SCLK
- U1 pad 36: (no net) -> MOSI
- U1 pad 38: (no net) -> MISO
- U1 pad 39: (no net) -> SCL
- U1 pad 40: (no net) -> RXD
- U1 pad 41: (no net) -> TXD
- U1 pad 42: (no net) -> SDA
- U1 pad 5: (no net) -> Net-(C22-Pad1)
- U1 pad 6: (no net) -> Net-(C22-Pad2)
- U1 pad 7: (no net) -> Net-(C24-Pad2)
- U1 pad 8: (no net) -> Net-(C24-Pad1)
- U1 pad 9: (no net) -> RESET
- U2 pad 1: +3V3 -> Net-(C12-Pad1)
- U2 pad 5: Vin -> Vraw
- U3 pad 6: Net-(D1-Pad1) -> nSTDBY
- U3 pad 7: Net-(D2-Pad1) -> nCHRG
- U5 pad 24: (no net) -> RTS
- U5 pad 25: (no net) -> RXD
- U5 pad 26: (no net) -> TXD
- U5 pad 28: (no net) -> DTR
- U5 pad 29: Net-(U5-Pad29) -> GND
- U5 pad 3: (no net) -> GND
- U5 pad 4: (no net) -> USB_DP
- U5 pad 5: (no net) -> USB_DM
- U5 pad 6: (no net) -> +3V3
- U5 pad 7: (no net) -> +3V3
- U5 pad 8: (no net) -> Vin
- U5 pad 9: (no net) -> Net-(R15-Pad2)
- U6 pad 1: PSRAM_CS -> +5V
- U6 pad 2: SIO1 -> Net-(L2-Pad2)
- U6 pad 3: SIO2 -> GND
- U6 pad 4: GND -> Net-(L2-Pad1)
- U6 pad 5: SIO0 -> Vraw_for_5v
- U6 pad 6: SCLK -> Net-(R9-Pad1)
- U6 pad 7: SIO3 -> Net-(R9-Pad1)
- U6 pad 8: VDD_SDIO -> Net-(R9-Pad1)
Routing:
- net +5V: track 0.00 -> 161.6 mm, vias 0 -> 1
- net MISO: track 0.00 -> 127.3 mm, vias 0 -> 1
- net Vstrong: track 0.00 -> 106.2 mm
- net SPI_CS0: track 0.00 -> 102.5 mm, vias 0 -> 1
- net SDA: track 0.00 -> 99.2 mm, vias 0 -> 2
- net MOSI: track 0.00 -> 98.0 mm, vias 0 -> 1
- net SCL: track 0.00 -> 95.1 mm
- net Vraw: track 34.8 -> 128.4 mm, vias 0 -> 5
- net Vin: track 2.02 -> 93.3 mm, vias 0 -> 3
- net SCLK: track 5.93 -> 92.6 mm, vias 0 -> 1
- net DISABLE_5v: track 0.00 -> 79.1 mm, vias 0 -> 4
- net SPI_CS1: track 0.00 -> 76.8 mm, vias 0 -> 1
- net IO3: track 0.00 -> 71.8 mm, vias 0 -> 1
- net IO2: track 0.00 -> 69.9 mm, vias 0 -> 1
- net GND: track 26.4 -> 96.0 mm, vias 0 -> 31
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- added copper zone on In2.Cu, net +3V3
- added copper zone on F.Cu, net GND
- added copper zone on In1.Cu, net GND
Other:
- board size 90 x 90 mm -> 90.3 x 95.8 mm

Commit message: routed
Parts:
- moved R12 42.8 mm to (87.2, 36.3)
- moved R13 42.8 mm to (89.2, 36.3)
- moved R14 32.6 mm to (72.3, 33.6), turned to 270 degrees
- moved R42 29.7 mm to (72.3, 35.6), turned to 270 degrees
- moved R8 17.3 mm to (84.0, 58.2), turned to 0 degrees
- moved C11 14.0 mm to (84.1, 55.7), turned to 0 degrees
- moved R1 12.4 mm to (84.1, 54.0), turned to 0 degrees
- moved U3 12.1 mm to (78.6, 57.6), turned to 180 degrees
- moved C15 9.61 mm to (102.2, 57.6), turned to 270 degrees
- moved R3 9.42 mm to (81.5, 44.6), turned to 270 degrees
- moved Q7 9.32 mm to (77.4, 49.0)
- moved R28 9.32 mm to (74.3, 49.8)
- moved R29 9.32 mm to (74.3, 47.5)
- moved Q8 9.32 mm to (82.1, 49.0)
- moved D1 9.32 mm to (78.4, 44.4)
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Connections:
- C14 pad 1: +3V3 -> Net-(C12-Pad1)
- J3 pad 1: Vcharge -> Vraw
- J3 pad 3: Vraw -> Vcharge
- U1 pad 10: ADC0 -> ADC1
- U1 pad 11: ADC1 -> ADC0
Routing:
- net ADC0: track 7.18 -> 56.9 mm, vias 0 -> 2
- net Vin: track 93.3 -> 43.8 mm, vias 3 -> 2
- net Vraw: track 128.4 -> 89.1 mm, vias 5 -> 2
- net ADC1: track 7.99 -> 40.3 mm, vias 0 -> 2
- net +5V: track 161.6 -> 130.2 mm, vias 1 -> 6
- net DISABLE_5v: track 79.1 -> 51.2 mm, vias 4 -> 0
- net SPI_CS0: track 102.5 -> 83.8 mm, vias 1 -> 2
- net GND: track 96.0 -> 113.3 mm, vias 31 -> 54
- net IO0: track 66.4 -> 83.1 mm, vias 2 -> 1
- net Vcharge: track 40.0 -> 56.2 mm, vias 0 -> 3
- net nCHRG: track 27.2 -> 12.1 mm, vias 0 -> 2
- net SPI_CS1: track 76.8 -> 89.9 mm, vias 1 -> 2
- net MISO_5v: track 21.9 -> 31.3 mm, vias 2 -> 0
- net MISO: track 127.3 -> 118.1 mm, vias 1 -> 3
- net +3V3: track 46.7 -> 56.0 mm, vias 19 -> 23
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Other:
- board size 90.3 x 95.8 mm -> 87 x 87 mm

Commit message: silkscreen
Other:
- board text added: "*"
- board text added: "+"
- board text added: "-"
- board text added: "1-2 normal 2-3 bypass regulators"
- board text added: "Boot0"
- board text added: "Charge"
- board text added: "J1: ext DC: 1.8 to 4.6v for Li recharge: 4.5 to 5.5v"
- board text added: "J3: 1-2 ext DC 2-3 Li recharge"
- board text added: "Reset"
- board text added: "Standby"
- board text added: "eboard 2020-12-06"
