File: eboard/eboard.kicad_pcb (KiCad board)
At the start: 4 copper layers, 87 x 87 mm, 132 parts, among them J1 Conn_01x02_Male, J10 Conn_01x06_Male, J11 Conn_01x02_Male, J12 Conn_01x02_Male, J13 Conn_01x02_Male, J14 Conn_01x02_Male, J15 Conn_01x02_Male, J16 Conn_01x03_Male, J17 Conn_01x03_Male, J18 Conn_01x03_Male, J19 Conn_01x03_Male, J2 USB_B_Micro, J20 Conn_01x02_Male, J21 Conn_01x03_Male, J3 Conn_01x03_Male, J4 jst_battery, J5 Conn_01x02_Male, J6 Conn_01x03_Male, J7 Conn_01x04_Male, J8 Conn_01x04_Male, J9 Conn_01x06_Male, Q1 AO4407A_new, Q10 BSS138K, Q11 AO4407A_new, Q12 BSS138K, Q13 BSS138K, Q14 BSS138K, Q15 BSS138K, Q16 BSS138K, Q17 BSS138K, Q18 AO4407A_new, Q19 AO4407A_new, Q2 S8050, Q20 AO4407A_new, Q3 S8050, Q4 BSS138K, Q5 BSS138K, Q6 AO4407A_new, Q7 BSS138K, Q8 BSS138K, Q9 BSS138K, SW1 pushbutton_switch, SW2 pushbutton_switch, U1 ESP32-PICO-D4, U2 TPS63000, U3 TP4056, U4 SRV05-4, U5 CP2102, U6 TPS63000, U7 SRV05-4, U8 SRV05-4, U9 SRV05-4

Commit message: lib
Parts:
- Q1, Q11, Q18, Q19, Q20, Q6: value AO4407A_new -> AO4407
Connections:
- H1 pad 1: (no net) -> GND
- H2 pad 1: (no net) -> GND
- H3 pad 1: (no net) -> GND
- H4 pad 1: (no net) -> GND
Changed lines of the file:
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@@
       (effects (font (size 1 1) (thickness 0.15)))
     )
-    (fp_text value AO4407A_new (at 0 3.4) (layer F.Fab)
+    (fp_text value AO4407 (at 0 3.4) (layer F.Fab)
       (effects (font (size 1 1) (thickness 0.15)))
     )
@@
       (effects (font (size 1 1) (thickness 0.15)))
     )
-    (fp_text value AO4407A_new (at 0 3.4 90) (layer F.Fab)
+    (fp_text value AO4407 (at 0 3.4 90) (layer F.Fab)
       (effects (font (size 1 1) (thickness 0.15)))
     )
@@
       (effects (font (size 1 1) (thickness 0.15)))
     )
-    (fp_text value AO4407A_new (at 0 3.4) (layer F.Fab)
+    (fp_text value AO4407 (at 0 3.4) (layer F.Fab)
       (effects (font (size 1 1) (thickness 0.15)))
     )
@@
       (effects (font (size 1 1) (thickness 0.15)))
     )
-    (fp_text value AO4407A_new (at 0 3.4) (layer F.Fab)
+    (fp_text value AO4407 (at 0 3.4) (layer F.Fab)
       (effects (font (size 1 1) (thickness 0.15)))
     )
@@
       (effects (font (size 1 1) (thickness 0.15)))
     )
-    (fp_text value AO4407A_new (at 0 3.4) (layer F.Fab)
+    (fp_text value AO4407 (at 0 3.4) (layer F.Fab)
       (effects (font (size 1 1) (thickness 0.15)))
     )
@@
       (effects (font (size 1 1) (thickness 0.15)))
     )
-    (fp_text value AO4407A_new (at 0 3.4) (layer F.Fab)
+    (fp_text value AO4407 (at 0 3.4) (layer F.Fab)
       (effects (font (size 1 1) (thickness 0.15)))
     )
@@
       (effects (font (size 1 1) (thickness 0.15)))
     )
-    (pad 1 np_thru_hole circle (at 0 0) (size 3.2 3.2) (drill 3.2) (layers *.Cu *.Mask))
+    (pad 1 np_thru_hole circle (at 0 0) (size 3.2 3.2) (drill 3.2) (layers *.Cu *.Mask)
+      (net 1 GND))
   )
   (module MountingHole:MountingHole_3.2mm_M3 (layer F.Cu)
@@
       (effects (font (size 1 1) (thickness 0.15)))
     )
-    (pad 1 np_thru_hole circle (at 0 0) (size 3.2 3.2) (drill 3.2) (layers *.Cu *.Mask))
+    (pad 1 np_thru_hole circle (at 0 0) (size 3.2 3.2) (drill 3.2) (layers *.Cu *.Mask)
+      (net 1 GND))
   )
   (module MountingHole:MountingHole_3.2mm_M3 (layer F.Cu)
@@
     (fp_circle (center 0 0) (end 3.2 0) (layer Cmts.User) (width 0.15))
     (fp_circle (center 0 0) (end 3.45 0) (layer F.CrtYd) (width 0.05))
-    (pad 1 np_thru_hole circle (at 0 0) (size 3.2 3.2) (drill 3.2) (layers *.Cu *.Mask))
+    (pad 1 np_thru_hole circle (at 0 0) (size 3.2 3.2) (drill 3.2) (layers *.Cu *.Mask)
+      (net 1 GND))
   )
   (module MountingHole:MountingHole_3.2mm_M3 (layer F.Cu)
@@
     (fp_circle (center 0 0) (end 3.2 0) (layer Cmts.User) (width 0.15))
     (fp_circle (center 0 0) (end 3.45 0) (layer F.CrtYd) (width 0.05))
-    (pad 1 np_thru_hole circle (at 0 0) (size 3.2 3.2) (drill 3.2) (layers *.Cu *.Mask))
+    (pad 1 np_thru_hole circle (at 0 0) (size 3.2 3.2) (drill 3.2) (layers *.Cu *.Mask)
+      (net 1 GND))
   )
   (module Capacitor_SMD:C_0402_1005Metric (layer F.Cu)

Commit message: ecos from v1
Parts:
- H1, H2, H3, H4: value MountingHole -> MountingHole_Pad; footprint MountingHole:MountingHole_3.2mm_M3 -> MountingHole:MountingHole_3.2mm_M3_Pad
Connections:
- R5 pad 1: Net-(R5-Pad1) -> Vraw
- R9 pad 1: Net-(R9-Pad1) -> Vraw_for_5v
- U2 pad 6: Net-(R5-Pad1) -> Vraw
- U2 pad 7: Net-(R5-Pad1) -> Vraw
- U2 pad 8: Net-(R5-Pad1) -> Vraw
- U5 pad 25: RXD -> TXD
- U5 pad 26: TXD -> RXD
- U6 pad 6: Net-(R9-Pad1) -> Vraw_for_5v
- U6 pad 7: Net-(R9-Pad1) -> Vraw_for_5v
- U6 pad 8: Net-(R9-Pad1) -> Vraw_for_5v
Routing:
- net Vraw_for_5v: track 16.9 -> 24.7 mm
- net Vraw: track 89.1 -> 96.6 mm
- net Net-(R9-Pad1): track 3.60 -> 0.00 mm
- net Net-(R5-Pad1): track 2.97 -> 0.00 mm
- net TXD: track 53.5 -> 54.9 mm
- net RXD: track 53.2 -> 52.6 mm

Commit message: remove 5v
Parts:
- removed C15, C18, C19, C8: 10u, Capacitor_SMD:C_0402_1005Metric
- removed C16: 100n, Capacitor_SMD:C_0402_1005Metric
- removed C17: 2.2pF, Capacitor_SMD:C_0402_1005Metric
- removed D5: SS210, Diode_SMD:D_SMA
- removed J10: Conn_01x06_Male, Connector_PinHeader_2.54mm:PinHeader_1x06_P2.54mm_Vertical
- removed J6: Conn_01x03_Male, Connector_PinHeader_2.54mm:PinHeader_1x03_P2.54mm_Vertical
- removed J8: Conn_01x04_Male, Connector_PinHeader_2.54mm:PinHeader_1x04_P2.54mm_Vertical
- removed L2: 2.2uH, Inductor_SMD:L_Coilcraft_XxL4020
- removed Q4, Q5: BSS138K, Package_TO_SOT_SMD:SOT-23
- removed Q6: AO4407, Package_SO:SOIC-8_3.9x4.9mm_P1.27mm
- removed R10: 1meg, Resistor_SMD:R_0603_1608Metric
- removed R11: 100k, Resistor_SMD:R_0402_1005Metric
- removed R21, R22, R23, R24, R25: 3.3k, Resistor_SMD:R_0402_1005Metric
- removed R26: 10k, Resistor_SMD:R_0402_1005Metric
- removed R27, R9: 100, Resistor_SMD:R_0402_1005Metric
- removed U6: TPS63000, Package_SON:Texas_DRC0010J_ThermalVias
- J21: value Conn_01x03_Male -> Conn_01x02_Male; footprint Connector_PinHeader_2.54mm:PinHeader_1x03_P2.54mm_Vertical -> Connector_PinHeader_2.54mm:PinHeader_1x02_P2.54mm_Vertical
- moved J21 0.54 mm to (49.2, 77.0)
Connections:
- C12 pad 1: Net-(C12-Pad1) -> +3V3
- C14 pad 1: Net-(C12-Pad1) -> +3V3
- R6 pad 1: Net-(C12-Pad1) -> +3V3
- U1 pad 22: DISABLE_5v -> (no net)
- U1 pad 29: SPI_CS1 -> (no net)
- U2 pad 1: Net-(C12-Pad1) -> +3V3
- U8 pad 3: SPI_CS1 -> (no net)
Routing:
- net +5V: track 130.2 -> 0.00 mm, vias 6 -> 0
- net SPI_CS1: track 89.9 -> 0.00 mm, vias 2 -> 0
- net DISABLE_5v: track 51.2 -> 0.00 mm
- net MISO_5v: track 31.3 -> 0.00 mm
- net Vraw_for_5v: track 24.7 -> 0.00 mm
- net Vraw: track 96.6 -> 75.2 mm
- net SCL_5v: track 21.0 -> 0.00 mm
- net SDA_5v: track 17.3 -> 0.00 mm
- net GND: track 113.3 -> 97.3 mm, vias 54 -> 52
- net Net-(C12-Pad1): track 15.1 -> 0.00 mm
- net MISO: track 118.1 -> 103.9 mm
- net +3V3: track 56.0 -> 46.8 mm, vias 23 -> 18
- net SCL: track 102.6 -> 94.1 mm, vias 3 -> 2
- net Net-(C17-Pad2): track 7.12 -> 0.00 mm
- net Net-(L2-Pad1): track 4.36 -> 0.00 mm
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Other:
- board text removed: "1-2 normal 2-3 bypass regulators"

Commit message: v2
Parts:
- removed Q7, Q8: BSS138K, Package_TO_SOT_SMD:SOT-23
- removed R28: 100, Resistor_SMD:R_0402_1005Metric
- removed R29: 100k, Resistor_SMD:R_0402_1005Metric
Connections:
- D1 pad 1: Net-(D1-Pad1) -> nCHRG
- D2 pad 1: Net-(D2-Pad1) -> nSTDBY
- U1 pad 28: ENABLE_STATUS -> (no net)
Routing:
- net ENABLE_STATUS: track 17.2 -> 0.00 mm
- net Net-(Q7-Pad1): track 9.72 -> 0.00 mm
- net Vcharge: track 56.2 -> 50.6 mm
- net nCHRG: track 12.1 -> 17.1 mm
- net Net-(D1-Pad1): track 3.74 -> 0.00 mm
- net Net-(D2-Pad1): track 3.52 -> 0.00 mm
- net nSTDBY: track 13.5 -> 16.5 mm
- net MISO: track 103.9 -> 101.8 mm, vias 3 -> 2
Other:
- board text added: "eboard 2021-02-20"
- board text removed: "eboard 2020-12-06"

Commit message: leds
Parts:
- D1: value ledgreen -> ledgreen_0805; footprint LED_SMD:LED_0603_1608Metric -> LED_SMD:LED_0805_2012Metric
- D4: value ledgreen -> ledyellow
- moved D1 0.76 mm to (78.4, 45.2)
- moved D4 0.32 mm to (64.0, 45.4)
Routing:
- net nCHRG: track 17.1 -> 15.7 mm
