File: eboard/eboard.sch (KiCad schematic (older format))
At the start: 41 parts, among them J1 Conn_01x02_Male, J2 USB_B_Micro, J3 Conn_01x03_Male, J4 Conn_01x02_Male, J5 Conn_01x02_Male, Q1 AO4407A, U1 ESP32-PICO-D4, U2 TPS63000, U3 TP4056, U4 SRV05-4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

Commit message: progress
Parts:
- removed C16: 100n, Capacitor_SMD:C_0402_1005Metric, symbol pace:100n
- removed U6: W25Q128JVSIQ, Package_SO:SOIC-8_5.23x5.23mm_P1.27mm, symbol pace:W25Q128JVSIQ
- added C?: 100n, Capacitor_SMD:C_0402_1005Metric, symbol pace:100n
- added D?: ledgreen, LED_SMD:LED_0603_1608Metric, symbol pace:ledgreen
- added Q? (x2): S8050, Package_TO_SOT_SMD:SOT-23, symbol pace:S8050
- added R? (x9): 10k, Resistor_SMD:R_0402_1005Metric, symbol pace:10k
- added SW? (x2): SW_Push, symbol Switch:SW_Push
Connections:
- net labels added: DTR, IO0, IO5, RESET, RTS, RXD, TXD
- net labels removed: PSRAM_CS, SCLK, SIO0, SIO1, SIO2, SIO3, VDD_SDIO
- wire segments 114 -> 161
- no-connect marks 3 -> 17
Other:
- note added: "boot option"
- note added: "external\nflash\n(not used)"
- note added: "input only"
- moved on the sheet: C1, C2, C3, C4, C5, C6, C7, U1, U5

Commit message: io
Parts:
- removed Q1: AO4407A, Package_SO:SOIC-8_3.9x4.9mm_P1.27mm, symbol pace:AO4407A
- added C16: 100n, Capacitor_SMD:C_0402_1005Metric, symbol pace:100n
- added C17: 2.2pF, Capacitor_SMD:C_0402_1005Metric, symbol pace:2.2pF
- added C18, C19, C8: 10u, Capacitor_SMD:C_0402_1005Metric, symbol pace:10u
- added J6: Conn_01x02_Male, symbol Connector:Conn_01x02_Male
- added L2: 2.2uH, Inductor_SMD:L_Coilcraft_XxL4020, symbol pace:2.2uH
- added Q1: AO4407A_new, Package_SO:SOIC-8_3.9x4.9mm_P1.27mm, symbol pace:AO4407A_new
- added R10: 1meg, Resistor_SMD:R_0603_1608Metric, symbol pace:1meg
- added R11: 180k, Resistor_SMD:R_0603_1608Metric, symbol pace:180k
- added R9: 100, Resistor_SMD:R_0402_1005Metric, symbol pace:100
- added U6: TPS63000, Package_SON:Texas_DRC0010J_ThermalVias, symbol pace:TPS63000
- gave numbers to parts that had none: 15
Connections:
- net labels added: +5V, MISO, MOSI, OUT0, OUT1, OUT2, OUT3, SCL, SCLK, SDA, SPI_CS
- wire segments 161 -> 199
- no-connect marks 17 -> 32
Other:
- moved on the sheet: C10, C11, C12, C13, C14, C15, C9, D1, D2, J3, J4, J5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

Commit message: power
Parts:
- removed J6: Conn_01x02_Male, symbol Connector:Conn_01x02_Male
- removed R1: 1meg, Resistor_SMD:R_0603_1608Metric, symbol pace:1meg
- removed R11: 180k, Resistor_SMD:R_0603_1608Metric, symbol pace:180k
- added Q? (x2): 2N7002, Package_TO_SOT_SMD:SOT-23, symbol pace:2N7002
- added Q?: AO4407A_new, Package_SO:SOIC-8_3.9x4.9mm_P1.27mm, symbol pace:AO4407A_new
- added R? (x3): 100k, Resistor_SMD:R_0402_1005Metric, symbol pace:100k
- added R? (x2): 100, Resistor_SMD:R_0402_1005Metric, symbol pace:100
- added R?: 10k, Resistor_SMD:R_0402_1005Metric, symbol pace:10k
Connections:
- net GND: now also R?.2, R?.2
- net Vraw: now also Q?.1 (S), Q?.2 (Sb), Q?.3 (Sc)
- net DISABLE_5v: now reaches U1.17 (IO14)
- net DISABLE_5v: now also R?.2
- net ENABLE_STATUS: now reaches U1.20 (IO13)
- net ENABLE_STATUS: now also R?.2
- net Vcharge: now reaches C11.1, J3.1 (Pin_1), R2.2, R3.1, R4.1, U3.4 (VCC), U3.8 (CE)
- net Vcharge: now also R?.1, R?.1
- net at D1.1 (K): now also Q?.3 (D); no longer U3.6 (~STDBY)
- net at D2.1 (K): now also Q?.3 (D); no longer U3.7 (~CHRG)
- net at C17.2, R10.2, U6.10 (FB): now also R?.1
- net Vraw_for_5v: now reaches C8.1, U6.5 (VIN)
- net Vraw_for_5v: now also Q?.5 (Dd), Q?.6 (Dc), Q?.7 (Db), Q?.8 (D)
- new net: Q?.1 (G), Q?.1 (G), R?.1, R?.2
- new net: Q?.4 (G), R?.1
- new net: R?.1, R?.2
- new net nCHRG: Q?.2 (S), U3.7 (~CHRG)
- new net nSTDBY: Q?.2 (S), U3.6 (~STDBY)
- no-connect marks 32 -> 30
Other:
- note added: "5.05v nominal\nwith 1% reisistors: 4.59 to 5.14v"
- note added: "Connect 1-2: lithium battery with recharge\nConnect 2-3: external DC supply (usb or header)"
- note added: "Diode drops 5v usb input\nto safe range for dc-dc converter,\nand prevents backdriving USB"
- note added: "If 5v desired,\nmin Vin TBD"
- note added: "led's enabled by default\nforced off by driving low"
- note removed: "Connect 1-2: lithium battery with recharge\nConnect 2-3: external DC supply"
- note removed: "Diode drops 5v usb input\nto safe range for dc-dc converter"
- moved on the sheet: C11, C13, D1, D2, J3, J4, J5, R2, R3, R4, R8, U3

Commit message: routing
Parts:
- removed J4: Conn_01x02_Male, Connector_PinHeader_2.54mm:PinHeader_1x02_P2.54mm_Vertical, symbol Connector:Conn_01x02_Male
- removed Q? (x2): 2N7002, Package_TO_SOT_SMD:SOT-23, symbol pace:2N7002
- removed R12, R13, R14: 10k, Resistor_SMD:R_0402_1005Metric, symbol pace:10k
- removed SW1, SW2: SW_Push, symbol Switch:SW_Push
- added C21: 100n, Capacitor_SMD:C_0402_1005Metric, symbol pace:100n
- added C22, C24: 330pF, Capacitor_SMD:C_0402_1005Metric, symbol pace:330pF
- added C23: 1u, Capacitor_SMD:C_0402_1005Metric, symbol pace:1u
- added H1, H2, H3, H4: MountingHole, MountingHole:MountingHole_3.2mm_M3, symbol Mechanical:MountingHole
- added J4: jst_battery, Connector_JST:JST_PH_B2B-PH-K_1x02_P2.00mm_Vertical, symbol pace:jst_battery
- added J6: Conn_01x03_Male, Connector_PinHeader_2.54mm:PinHeader_1x03_P2.54mm_Vertical, symbol Connector:Conn_01x03_Male
- added Q7, Q8: BSS138K, Package_TO_SOT_SMD:SOT-23, symbol pace:BSS138K
- added R12, R13, R14, R42: 100k, Resistor_SMD:R_0402_1005Metric, symbol pace:100k
- added SW1, SW2: pushbutton_switch, Button_Switch_THT:SW_PUSH_6mm, symbol pace:pushbutton_switch
- gave numbers to parts that had none: 7
Connections:
- net SPI_CS is gone; now on net OUT2: U1.14 (IO25)
- net +3V3: now also C21.1, C23.1, J6.2 (Pin_2); no longer C12.1, R6.1, U2.1 (VOUT)
- net DISABLE_5v: now also U1.22 (IO2); no longer U1.17 (IO14)
- net ENABLE_STATUS: now also U1.28 (SD2/IO9); no longer U1.20 (IO13)
- net GND: now also C21.2, C23.2, J4.2 (Pin_2), J6.3 (Pin_3), R13.2, R42.2, SW1.1, SW2.1
- net IO0: now also U1.24 (IO4); no longer Q3.3 (C), R20.2, U1.23 (IO0)
- net OUT0: now also U1.17 (IO14); no longer U1.15 (IO26)
- net OUT2: no longer U1.12 (IO32)
- net RESET: now also SW1.2
- net Vin: now also U5.8 (VBUS), R12.1
- net Vraw: now also J4.1 (Pin_1), R14.1
- net nCHRG: now also Q7.2 (S)
- net nSTDBY: now also Q8.2 (S)
- net ADC0: now reaches U1.10 (IO34)
- net ADC0: now also R12.2, R13.1
- net ADC1: now reaches U1.11 (IO35)
- net ADC1: now also R14.2, R42.1
- net IO2: now reaches U1.18 (IO12)
- net WIFI: now reaches U1.2 (LNA_IN)
- net SPI_CS0: now reaches U1.21 (IO15)
- net SPI_CS1: now reaches U1.29 (SD3/IO10)
- net at U1.5 (SENSOR_VP): now also C22.1
- net at U1.6 (SENSOR_CAPP): now also C22.2
- net at U1.7 (SENSOR_CAPN): now also C24.2
- net at U1.8 (SENSOR_VN): now also C24.1
- net at D2.1 (K): now also Q8.3 (D)
- net at D1.1 (K): now also Q7.3 (D)
- net at R28.1, R29.2: now also Q7.1 (G), Q8.1 (G)
- net IO5 renamed STATUS_LED
- new net: C12.1, J6.1 (Pin_1), R6.1, U2.1 (VOUT)
- new net BOOT0: Q3.3 (C), R20.2, SW2.2, U1.23 (IO0)
- new net IO1: U1.20 (IO13)
- new net IO3: U1.15 (IO26)
- no-connect marks 30 -> 18
Other:
- note added: "external\nflash\n(used inside pico module?)\n"
- note added: "strapping"
- note added: "temporary header\nin case power supply\ndoesn't work\n"
- note removed: "If 5v desired,\nmin Vin TBD"
- note removed: "boot option"
- note removed: "external\nflash\n(not used)"
- moved on the sheet: C14, C15

Commit message: routed
Connections:
- net +3V3: no longer C14.1
- net ADC0: now also U1.11 (IO35); no longer U1.10 (IO34)
- net ADC1: now also U1.10 (IO34); no longer U1.11 (IO35)
- net Vcharge: now also J3.3 (Pin_3); no longer J3.1 (Pin_1)
- net Vraw: now also J3.1 (Pin_1); no longer J3.3 (Pin_3)
- net at C12.1, J6.1 (Pin_1), R6.1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: now also C14.1
Other:
- moved on the sheet: C12, C14, R6, R7
Changed lines of the file:
@@
 F 3 "~" H 2200 2550 50  0001 C CNN
 	1    2200 2550
-	0    -1   -1   0
+	0    1    -1   0
 $EndComp
 Text GLabel 1900 2150 0    50   Input ~ 0
@@
 L pace:1meg R6
 U 1 1 5FA96672
-P 3000 4800
-F 0 "R6" H 3059 4846 50  0000 L CNN
-F 1 "1meg" H 3059 4755 50  0000 L CNN
-F 2 "Resistor_SMD:R_0603_1608Metric" H 3000 4800 50  0001 C CNN
-F 3 "https://lcsc.com/product-detail/Chip-Resistor-Surface-Mount_Uniroyal-Elec-0603WAF1004T5E_C22935.html/?href=jlc-SMT" H 3000 4800 50  0001 C CNN
-F 4 "C22935" H 3000 4800 50  0001 C CNN "LCSC"
-	1    3000 4800
+P 2900 4800
+F 0 "R6" H 2959 4846 50  0000 L CNN
+F 1 "1meg" H 2959 4755 50  0000 L CNN
+F 2 "Resistor_SMD:R_0603_1608Metric" H 2900 4800 50  0001 C CNN
+F 3 "https://lcsc.com/product-detail/Chip-Resistor-Surface-Mount_Uniroyal-Elec-0603WAF1004T5E_C22935.html/?href=jlc-SMT" H 2900 4800 50  0001 C CNN
+F 4 "C22935" H 2900 4800 50  0001 C CNN "LCSC"
+	1    2900 4800
 	1    0    0    -1
 $EndComp
@@
 L pace:180k R7
 U 1 1 5FA97E48
-P 3000 5100
-F 0 "R7" H 3059 5146 50  0000 L CNN
-F 1 "180k" H 3059 5055 50  0000 L CNN
-F 2 "Resistor_SMD:R_0603_1608Metric" H 3000 5100 50  0001 C CNN
-F 3 "https://lcsc.com/product-detail/Chip-Resistor-Surface-Mount_Uniroyal-Elec-0603WAF1803T5E_C22827.html/?href=jlc-SMT" H 3000 5100 50  0001 C CNN
-F 4 "C22827" H 3000 5100 50  0001 C CNN "LCSC"
-	1    3000 5100
-	1    0    0    -1
-$EndComp
-Wire Wire Line
-	2600 4650 3000 4650
-Wire Wire Line
-	3000 4650 3000 4700
-Wire Wire Line
-	3000 4900 3000 4950
+P 2900 5100
+F 0 "R7" H 2959 5146 50  0000 L CNN
+F 1 "180k" H 2959 5055 50  0000 L CNN
+F 2 "Resistor_SMD:R_0603_1608Metric" H 2900 5100 50  0001 C CNN
+F 3 "https://lcsc.com/product-detail/Chip-Resistor-Surface-Mount_Uniroyal-Elec-0603WAF1803T5E_C22827.html/?href=jlc-SMT" H 2900 5100 50  0001 C CNN
+F 4 "C22827" H 2900 5100 50  0001 C CNN "LCSC"
+	1    2900 5100
+	1    0    0    -1
+$EndComp
+Wire Wire Line
+	2600 4650 2900 4650
+Wire Wire Line
+	2900 4650 2900 4700
+Wire Wire Line
+	2900 4900 2900 4950
 $Comp
 L power:GND #PWR?
 U 1 1 5FAA312D
-P 3000 5200
-F 0 "#PWR?" H 3000 4950 50  0001 C CNN
-F 1 "GND" H 3005 5027 50  0000 C CNN
-F 2 "" H 3000 5200 50  0001 C CNN
-F 3 "" H 3000 5200 50  0001 C CNN
-	1    3000 5200
-	1    0    0    -1
-$EndComp
-Wire Wire Line
-	2600 4850 2800 4850
-Wire Wire Line
-	2800 4850 2800 4950
-Wire Wire Line
-	2800 4950 3000 4950
-Connection ~ 3000 4950
-Wire Wire Line
-	3000 4950 3000 5000
+P 2900 5200
+F 0 "#PWR?" H 2900 4950 50  0001 C CNN
+F 1 "GND" H 2905 5027 50  0000 C CNN
+F 2 "" H 2900 5200 50  0001 C CNN
+F 3 "" H 2900 5200 50  0001 C CNN
+	1    2900 5200
+	1    0    0    -1
+$EndComp
+Wire Wire Line
+	2600 4850 2750 4850
+Wire Wire Line
+	2750 4850 2750 4950
+Wire Wire Line
+	2750 4950 2900 4950
+Connection ~ 2900 4950
+Wire Wire Line
+	2900 4950 2900 5000
 Text Notes 2600 5700 0    50   ~ 0
 3.28v nominal\nwith 1% reisistors: 3.00 to 3.33v
@@
 L pace:2.2pF C12
 U 1 1 5FAAD83F
-P 3400 4800
-F 0 "C12" H 3492 4846 50  0000 L CNN
-F 1 "2.2pF" H 3492 4755 50  0000 L CNN
-F 2 "Capacitor_SMD:C_0402_1005Metric" H 3400 4800 50  0001 C CNN
-F 3 "https://lcsc.com/product-detail/Multilayer-Ceramic-Capacitors-MLCC-SMD-SMT_2-2pF-2R2-0-25pF-50V_C1559.html/?href=jlc-SMT" H 3400 4800 50  0001 C CNN
-F 4 "C1559" H 3400 4800 50  0001 C CNN "LCSC"
-	1    3400 4800
-	1    0    0    -1
-$EndComp
-Wire Wire Line
-	3000 4650 3400 4650
-Wire Wire Line
-	3400 4650 3400 4700
-Connection ~ 3000 4650
-Wire Wire Line
-	3000 4950 3400 4950
-Wire Wire Line
-	3400 4950 3400 4900
+P 3250 4800
+F 0 "C12" H 3342 4846 50  0000 L CNN
+F 1 "2.2pF" H 3342 4755 50  0000 L CNN
+F 2 "Capacitor_SMD:C_0402_1005Metric" H 3250 4800 50  0001 C CNN
+F 3 "https://lcsc.com/product-detail/Multilayer-Ceramic-Capacitors-MLCC-SMD-SMT_2-2pF-2R2-0-25pF-50V_C1559.html/?href=jlc-SMT" H 3250 4800 50  0001 C CNN
+F 4 "C1559" H 3250 4800 50  0001 C CNN "LCSC"
+	1    3250 4800
+	1    0    0    -1
+$EndComp
+Wire Wire Line
+	2900 4650 3250 4650
+Wire Wire Line
+	3250 4650 3250 4700
+Connection ~ 2900 4650
+Wire Wire Line
+	2900 4950 3250 4950
+Wire Wire Line
+	3250 4950 3250 4900
 $Comp
 L pace:10u C14
 U 1 1 5FAB3458
-P 4250 5000
-F 0 "C14" H 4342 5046 50  0000 L CNN
-F 1 "10u" H 4342 4955 50  0000 L CNN
-F 2 "Capacitor_SMD:C_0402_1005Metric" H 4250 5000 50  0001 C CNN
-F 3 "https://datasheet.lcsc.com/szlcsc/Samsung-Electro-Mechanics-CL05A106MQ5NUNC_C15525.pdf" H 4250 5000 50  0001 C CNN
-F 4 "C15525" H 4250 5000 50  0001 C CNN "LCSC"
-	1    4250 5000
-	1    0    0    -1
-$EndComp
-Wire Wire Line
-	4250 4850 4250 4900
+P 3650 5100
+F 0 "C14" H 3742 5146 50  0000 L CNN
+F 1 "10u" H 3742 5055 50  0000 L CNN
+F 2 "Capacitor_SMD:C_0402_1005Metric" H 3650 5100 50  0001 C CNN
+F 3 "https://datasheet.lcsc.com/szlcsc/Samsung-Electro-Mechanics-CL05A106MQ5NUNC_C15525.pdf" H 3650 5100 50  0001 C CNN
+F 4 "C15525" H 3650 5100 50  0001 C CNN "LCSC"
+	1    3650 5100
+	1    0    0    -1
+$EndComp
 $Comp
 L power:GND #PWR?
 U 1 1 5FAB6079
-P 4250 5100
-F 0 "#PWR?" H 4250 4850 50  0001 C CNN
-F 1 "GND" H 4255 4927 50  0000 C CNN
-F 2 "" H 4250 5100 50  0001 C CNN
-F 3 "" H 4250 5100 50  0001 C CNN
-	1    4250 5100
+P 3650 5200
+F 0 "#PWR?" H 3650 4950 50  0001 C CNN
+F 1 "GND" H 3655 5027 50  0000 C CNN
+F 2 "" H 3650 5200 50  0001 C CNN
+F 3 "" H 3650 5200 50  0001 C CNN
+	1    3650 5200
 	1    0    0    -1
 $EndComp
@@
 	1    0    0    -1
 $EndComp
-Wire Wire Line
-	4250 4850 4550 4850
 Wire Wire Line
 	4550 4850 4550 4700
@@
 Wire Wire Line
 	4000 4850 4150 4850
-Connection ~ 4250 4850
 Wire Wire Line
 	4000 4750 4000 4650
 Wire Wire Line
-	4000 4650 3400 4650
-Connection ~ 3400 4650
+	4000 4650 3650 4650
+Connection ~ 3250 4650
 Text Notes 3650 4400 0    50   ~ 0
 temporary header\nin case power supply\ndoesn't work\n
@@
 $EndComp
 Connection ~ 4150 4850
-Wire Wire Line
-	4150 4850 4250 4850
 Text GLabel 9650 2500 2    50   Input ~ 0
 SPI_CS1
@@
 Wire Wire Line
 	7500 2000 8050 2000
+Text GLabel 9650 4100 2    50   Input ~ 0
+ADC0
 Text GLabel 9650 4000 2    50   Input ~ 0
-ADC0
-Text GLabel 9650 4100 2    50   Input ~ 0
 ADC1
 $Comp
@@
 Text GLabel 9650 2700 2    50   Input ~ 0
 IO1
+Wire Wire Line
+	4150 4850 4550 4850
+Wire Wire Line
+	3650 5000 3650 4650
+Connection ~ 3650 4650
+Wire Wire Line
+	3650 4650 3250 4650
 $EndSCHEMATC

Commit message: silkscreen
Other:
- note added: "Connect 1-2: external DC supply (usb or header)\nConnect 2-3: lithium battery with recharge"
- note removed: "Connect 1-2: lithium battery with recharge\nConnect 2-3: external DC supply (usb or header)"
Changed lines of the file:
@@
 dc-dc converter / regulator
 Text Notes 2350 2250 0    50   ~ 0
-Connect 1-2: lithium battery with recharge\nConnect 2-3: external DC supply (usb or header)
+Connect 1-2: external DC supply (usb or header)\nConnect 2-3: lithium battery with recharge
 Wire Wire Line
 	4650 700  4500 700

Commit message: fab3
Parts:
- U2, U6: LCSC (none) -> C24966
Changed lines of the file:
@@
 F 2 "Package_SON:Texas_DRC0010J_ThermalVias" H 3050 4300 50  0001 C CNN
 F 3 "http://www.ti.com/lit/ds/symlink/tps63000.pdf" H 1900 5400 50  0001 C CNN
+F 4 "C24966" H 2200 4850 50  0001 C CNN "LCSC"
 	1    2200 4850
 	1    0    0    -1
@@
 F 2 "Package_SON:Texas_DRC0010J_ThermalVias" H 3000 6450 50  0001 C CNN
 F 3 "http://www.ti.com/lit/ds/symlink/tps63000.pdf" H 1850 7550 50  0001 C CNN
+F 4 "C24966" H 2150 7000 50  0001 C CNN "LCSC"
 	1    2150 7000
 	1    0    0    -1

Commit message: lib
Parts:
- H1, H2, H3, H4: symbol Mechanical:MountingHole -> pace:MountingHole_Pad
- J1, J5: symbol Connector:Conn_01x02_Male -> pace:Conn_01x02_Male
- J2: symbol Connector:USB_B_Micro -> pace:USB_B_Micro
- J3, J6: symbol Connector:Conn_01x03_Male -> pace:Conn_01x03_Male
- Q1, Q6: value AO4407A_new -> AO4407; symbol pace:AO4407A_new -> pace:AO4407
Connections:
- net GND: now also H1.1, H2.1, H3.1, H4.1
