File: eboard/io.sch (KiCad schematic (older format))
At the start: 51 parts, among them J10 Conn_01x06_Male, J11 Conn_01x02_Male, J12 Conn_01x02_Male, J13 Conn_01x02_Male, J14 Conn_01x02_Male, J15 Conn_01x02_Male, J16 Conn_01x03_Male, J17 Conn_01x03_Male, J18 Conn_01x03_Male, J19 Conn_01x03_Male, J20 Conn_01x02_Male, J21 Conn_01x03_Male, J7 Conn_01x04_Male, J8 Conn_01x04_Male, J9 Conn_01x06_Male, Q10 BSS138K, Q11 AO4407A_new, Q12 BSS138K, Q13 BSS138K, Q14 BSS138K, Q15 BSS138K, Q16 BSS138K, Q17 BSS138K, Q18 AO4407A_new, Q19 AO4407A_new, Q20 AO4407A_new, Q4 BSS138K, Q5 BSS138K, Q9 BSS138K, U7 SRV05-4, U8 SRV05-4, U9 SRV05-4

Commit message: lib
Parts:
- Q11, Q18, Q19, Q20: value AO4407A_new -> AO4407; symbol pace:AO4407A_new -> pace:AO4407
Changed lines of the file:
@@
 $EndComp
 $Comp
-L pace:AO4407A_new Q11
+L pace:AO4407 Q11
 U 1 1 5FEF36A8
 P 9550 1250
 F 0 "Q11" H 9900 1200 50  0000 L CNN
-F 1 "AO4407A_new" H 9900 1300 50  0000 L CNN
+F 1 "AO4407" H 9900 1300 50  0000 L CNN
 F 2 "Package_SO:SOIC-8_3.9x4.9mm_P1.27mm" H 9750 1350 50  0001 C CNN
 F 3 "https://jlcpcb.com/parts/componentSearch?searchTxt=ao4407" H 9550 1250 50  0001 C CNN
@@
 	7900 1900 8050 1900
 $Comp
-L pace:AO4407A_new Q20
+L pace:AO4407 Q20
 U 1 1 5FD6EF8A
 P 9500 2950
 F 0 "Q20" H 9850 2900 50  0000 L CNN
-F 1 "AO4407A_new" H 9850 3000 50  0000 L CNN
+F 1 "AO4407" H 9850 3000 50  0000 L CNN
 F 2 "Package_SO:SOIC-8_3.9x4.9mm_P1.27mm" H 9700 3050 50  0001 C CNN
 F 3 "https://jlcpcb.com/parts/componentSearch?searchTxt=ao4407" H 9500 2950 50  0001 C CNN
@@
 	7850 3600 8000 3600
 $Comp
-L pace:AO4407A_new Q19
+L pace:AO4407 Q19
 U 1 1 5FD77284
 P 9350 4750
 F 0 "Q19" H 9700 4700 50  0000 L CNN
-F 1 "AO4407A_new" H 9700 4800 50  0000 L CNN
+F 1 "AO4407" H 9700 4800 50  0000 L CNN
 F 2 "Package_SO:SOIC-8_3.9x4.9mm_P1.27mm" H 9550 4850 50  0001 C CNN
 F 3 "https://jlcpcb.com/parts/componentSearch?searchTxt=ao4407" H 9350 4750 50  0001 C CNN
@@
 	7700 5400 7850 5400
 $Comp
-L pace:AO4407A_new Q18
+L pace:AO4407 Q18
 U 1 1 5FD772D6
 P 9300 6450
 F 0 "Q18" H 9650 6400 50  0000 L CNN
-F 1 "AO4407A_new" H 9650 6500 50  0000 L CNN
+F 1 "AO4407" H 9650 6500 50  0000 L CNN
 F 2 "Package_SO:SOIC-8_3.9x4.9mm_P1.27mm" H 9500 6550 50  0001 C CNN
 F 3 "https://jlcpcb.com/parts/componentSearch?searchTxt=ao4407" H 9300 6450 50  0001 C CNN

Commit message: remove 5v
Parts:
- removed D5: SS210, Diode_SMD:D_SMA, symbol pace:SS210
- removed J10: Conn_01x06_Male, Connector_PinHeader_2.54mm:PinHeader_1x06_P2.54mm_Vertical, symbol Connector:Conn_01x06_Male
- removed J21: Conn_01x03_Male, Connector_PinHeader_2.54mm:PinHeader_1x03_P2.54mm_Vertical, symbol Connector:Conn_01x03_Male
- removed J8: Conn_01x04_Male, Connector_PinHeader_2.54mm:PinHeader_1x04_P2.54mm_Vertical, symbol Connector:Conn_01x04_Male
- removed Q4, Q5: BSS138K, Package_TO_SOT_SMD:SOT-23, symbol pace:BSS138K
- removed R21, R22, R23, R24, R25: 3.3k, Resistor_SMD:R_0402_1005Metric, symbol pace:3.3k
- added J21: Conn_01x02_Male, Connector_PinHeader_2.54mm:PinHeader_1x02_P2.54mm_Vertical, symbol pace:Conn_01x02_Male
Connections:
- net +3V3: now also J21.1 (Pin_1)
- net Vstrong: now also J21.2 (Pin_2)
- net SPI_CS1: no longer names the net of U8.3 (IO2)
- no-connect marks 1 -> 2
Other:
- note added: "open for external Vstrong\nelse jumper\n"
- note removed: "open for external Vstrong\nelse jumper middle to 3.3 or 5"

Commit message: v2a
Parts:
- Q11, Q18, Q19, Q20: LCSC C16072 -> C469397
Changed lines of the file:
@@
 F 2 "Package_SO:SOIC-8_3.9x4.9mm_P1.27mm" H 9750 1350 50  0001 C CNN
 F 3 "https://jlcpcb.com/parts/componentSearch?searchTxt=ao4407" H 9550 1250 50  0001 C CNN
-F 4 "C16072" H 9550 1250 50  0001 C CNN "LCSC"
+F 4 "C469397" H 9550 1250 50  0001 C CNN "LCSC"
 	1    9550 1250
 	1    0    0    1
@@
 F 2 "Package_SO:SOIC-8_3.9x4.9mm_P1.27mm" H 9700 3050 50  0001 C CNN
 F 3 "https://jlcpcb.com/parts/componentSearch?searchTxt=ao4407" H 9500 2950 50  0001 C CNN
-F 4 "C16072" H 9500 2950 50  0001 C CNN "LCSC"
+F 4 "C469397" H 9500 2950 50  0001 C CNN "LCSC"
 	1    9500 2950
 	1    0    0    1
@@
 F 2 "Package_SO:SOIC-8_3.9x4.9mm_P1.27mm" H 9550 4850 50  0001 C CNN
 F 3 "https://jlcpcb.com/parts/componentSearch?searchTxt=ao4407" H 9350 4750 50  0001 C CNN
-F 4 "C16072" H 9350 4750 50  0001 C CNN "LCSC"
+F 4 "C469397" H 9350 4750 50  0001 C CNN "LCSC"
 	1    9350 4750
 	1    0    0    1
@@
 F 2 "Package_SO:SOIC-8_3.9x4.9mm_P1.27mm" H 9500 6550 50  0001 C CNN
 F 3 "https://jlcpcb.com/parts/componentSearch?searchTxt=ao4407" H 9300 6450 50  0001 C CNN
-F 4 "C16072" H 9300 6450 50  0001 C CNN "LCSC"
+F 4 "C469397" H 9300 6450 50  0001 C CNN "LCSC"
 	1    9300 6450
 	1    0    0    1
